File: USB3Board.kicad_sch (KiCad schematic)
At the start: 6 parts, among them IC1 FT600Q-B-T, J1 USB_C_Receptacle, J2 Conn_02x20_Odd_Even, U1 TPD2EUSB30, U2 TPD2EUSB30, U3 TPD2EUSB30

Commit message: 1st pass
Parts:
- removed J1: USB_C_Receptacle, symbol Connector:USB_C_Receptacle
- removed J2: Conn_02x20_Odd_Even, symbol Connector_Generic:Conn_02x20_Odd_Even
- added C1, C10, C12, C14, C16, C18, C2, C20, C22, C3, C6, C7, C8, C9: 0.1uF, Capacitor_SMD:C_0402_1005Metric, symbol Device:C_Small
- added C24: 1uF, Capacitor_SMD:C_0402_1005Metric, symbol Device:C_Small
- added C25: 4.7uF, Capacitor_SMD:C_0402_1005Metric, symbol Device:C_Small
- added C4, C5: 18pF, Capacitor_SMD:C_0402_1005Metric, symbol Device:C_Small
- added D1, D2, D3: LED, LED_SMD:LED_0603_1608Metric, symbol Device:LED
- added H1: PM254-2-20-WS-8.5, EasyEDA:HDR-SMD_40P-P2.54_PM254-2-20-WS-8.5, symbol easyeda:PM254-2-20-WS-8.5
- added R1, R3, R4, R5: 100R, Resistor_SMD:R_0402_1005Metric, symbol Device:R
- added R10, R12, R13: 510R, Resistor_SMD:R_0402_1005Metric, symbol Device:R
- added R11, R9: 1K, Resistor_SMD:R_0402_1005Metric, symbol Device:R
- added R2: 33R, Resistor_SMD:R_0402_1005Metric, symbol Device:R
- added R6, R7: 5.1K, Resistor_SMD:R_0402_1005Metric, symbol Device:R
- added R8: 1.6K, Resistor_SMD:R_0402_1005Metric, symbol Device:R
- added RN1, RN2: 33R, EasyEDA:RES-ARRAY-SMD_0402-16P-L4.0-W1.6-BL, symbol Device:R_Pack08
- added RN3: 33R, EasyEDA:RES-ARRAY-SMD_0402-16P-L4.0-W1.6-BL, symbol Device:R_Pack08_Split
- added USB1: GT-USB-7001B, EasyEDA:USB-C-SMD_GT-USB-7001B, symbol easyeda:GT-USB-7001B
- added Y1: 30Mhz, Crystal:Crystal_SMD_TXC_AX_8045-2Pin_8.0x4.5mm, symbol Device:Crystal
- IC1: footprint FT600Q-B-T:QFN40P700X700X85-57N -> USBBoard3:QFN40P700X700X85-57N; LCSC Part (none) -> C3227923
- U1, U2, U3: LCSC Part (none) -> C97502
Connections:
- net +1V0: now reaches IC1.1 (AVDD)
- net +1V0: now also IC1.23 (VD10), IC1.26 (VD10), IC1.31 (DV10), IC1.37 (VD10), IC1.50 (VD10), C16.1, C18.1, C20.1, C22.1, C24.1, C25.1
- net at IC1.10 (~{RESET_N}): now also R5.1
- net at IC1.11 (~{WAKEUP_N}): now also R4.1
- net at IC1.12 (GPIO0): now also R1.1
- net at IC1.13 (GPIO1): now also R3.1
- net +3.3V: now reaches IC1.15 (VCC33)
- net +3.3V: now also IC1.19 (VCC33), IC1.22 (VDDA), IC1.30 (VCC33), IC1.38 (VCCIO), IC1.44 (VCCIO), IC1.52 (VCCIO), C10.1, C12.1, C14.1, C6.1, C7.1, C8.1, C9.1, H1.35, R10.2
- net XI: now reaches IC1.16 (XI)
- net XI: now also C5.1, Y1.1
- net XO: now reaches IC1.17 (XO)
- net XO: now also C4.1, Y1.2
- net USB_DP: now reaches IC1.18 (DP)
- net USB_DP: now also U1.1 (D+), USB1.A6 (DP1), USB1.B6 (DP2)
- net at IC1.2 (BE_0): now also RN3.16 (R1.2)
- net USB_DN: now reaches IC1.20 (DM)
- net USB_DN: now also U1.2 (D-), USB1.A7 (DN1), USB1.B7 (DN2)
- net at IC1.21 (RREF): now also R8.2
- net USB_TXN: now reaches IC1.24 (TODN)
- net USB_TXN: now also C1.2
- net USB_TXP: now reaches IC1.25 (TODP)
- net USB_TXP: now also C2.2
- net USB_RXN: now reaches IC1.27 (RIDN)
- net USB_RXN: now also U2.2 (D-), USB1.B10 (SSRXN1)
- net USB_RXP: now reaches IC1.28 (RIDP)
- net USB_RXP: now also U2.1 (D+), USB1.B11 (SSRXP1)
- net VBUS_IO: now reaches IC1.29 (VBUS)
- net VBUS_IO: now also R11.2, R12.1
- net at IC1.3 (BE_1): now also RN3.15 (R2.2)
- net GND: now reaches IC1.32 (GND)
- net GND: now also IC1.49 (GND), IC1.51 (GND), IC1.PAD (GND), U1.3 (GND), U2.3 (GND), U3.3 (GND), C10.2, C12.2, C14.2, C16.2, C18.2, C20.2, C22.2, C24.2, C25.2, C3.2, C4.2, C5.2, C6.2, C7.2, C8.2, C9.2, D1.1 (K), D2.1 (K), D3.1 (K), H1.15, H1.6, R11.1, R6.1, R7.2, R8.1, USB1.25 (SHELL), USB1.26 (SHELL), USB1.27 (SHELL), USB1.28 (SHELL), USB1.A1 (GND), USB1.A12 (GND), USB1.B1 (GND), USB1.B12 (GND)
- net at IC1.33 (DATA_0): now also RN2.8 (R8.1)
- net at IC1.34 (DATA_1): now also RN2.7 (R7.1)
- net at IC1.35 (DATA_2): now also RN2.6 (R6.1)
- net at IC1.36 (DATA_3): now also RN2.5 (R5.1)
- net at IC1.39 (DATA_4): now also RN2.4 (R4.1)
- net at IC1.4 (TXE_N): now also RN3.14 (R3.2)
- net at IC1.40 (DATA_5): now also RN2.3 (R3.1)
- net at IC1.41 (DATA_6): now also RN2.2 (R2.1)
- net at IC1.42 (DATA_7): now also RN2.1 (R1.1)
- net at IC1.43 (CLK): now also R2.1
- net at IC1.45 (DATA_8): now also RN1.8 (R8.1)
- net at IC1.46 (DATA_9): now also RN1.7 (R7.1)
- net at IC1.47 (DATA_10): now also RN1.6 (R6.1)
- net at IC1.48 (DATA_11): now also RN1.5 (R5.1)
- net at IC1.5 (RXF_N): now also RN3.13 (R4.2)
- net at IC1.53 (DATA_12): now also RN1.4 (R4.1)
- net at IC1.54 (DATA_13): now also RN1.3 (R3.1)
- net at IC1.55 (DATA_14): now also RN1.2 (R2.1)
- net at IC1.56 (DATA_15): now also RN1.1 (R1.1)
- net at IC1.6 (SIWU_N): now also RN3.12 (R5.2)
- net at IC1.7 (WR_N): now also RN3.11 (R6.2)
- net at IC1.8 (RD_N): now also RN3.10 (R7.2)
- net at IC1.9 (OE_N): now also RN3.9 (R8.2)
- net USB_I_TXP: now reaches U3.1 (D+)
- net USB_I_TXP: now also C2.1, USB1.A2 (SSTXP1)
- net USB_I_TXN: now reaches U3.2 (D-)
- net USB_I_TXN: now also C1.1, USB1.A3 (SSTXN1)
- new net: R7.1, USB1.B5 (CC2)
- new net: D1.2 (A), R9.1
- new net: R6.2, USB1.A5 (CC1)
- new net: D2.2 (A), R10.1
- new net: D3.2 (A), R13.1
- new net +5V: H1.26
- new net BE_0: H1.4, RN3.1 (R1.1)
- new net BE_1: H1.37, RN3.2 (R2.1)
- new net DATA0: H1.25, RN2.9 (R8.2)
- new net DATA1: H1.14, RN2.10 (R7.2)
- new net DATA10: H1.8, RN1.11 (R6.2)
- new net DATA11: H1.33, RN1.12 (R5.2)
- new net DATA12: H1.7, RN1.13 (R4.2)
- new net DATA13: H1.34, RN1.14 (R3.2)
- new net DATA14: H1.5, RN1.15 (R2.2)
- new net DATA15: H1.36, RN1.16 (R1.2)
- new net DATA2: H1.27, RN2.11 (R6.2)
- new net DATA3: H1.13, RN2.12 (R5.2)
- new net DATA4: H1.28, RN2.13 (R4.2)
- new net DATA5: H1.12, RN2.14 (R3.2)
- new net DATA6: H1.29, RN2.15 (R2.2)
- new net DATA7: H1.11, RN2.16 (R1.2)
- new net DATA8: H1.9, RN1.9 (R8.2)
- new net DATA9: H1.32, RN1.10 (R7.2)
- new net DATA_CLK: H1.30, R2.2
- new net GPIO0: H1.24, R1.2
- new net GPIO1: H1.16, R3.2
- new net INFO_LED: H1.21, R13.2
- new net VBUS: C3.1, R12.2, R9.2, USB1.A4 (VBUS), USB1.A9 (VBUS), USB1.B4 (VBUS), USB1.B9 (VBUS)
- new net ~{OE}: H1.40, RN3.8 (R8.1)
- new net ~{RD}: H1.1, RN3.7 (R7.1)
- new net ~{RESET}: H1.23, R5.2
- new net ~{RXF}: H1.38, RN3.4 (R4.1)
- new net ~{SIWU}: H1.2, RN3.5 (R5.1)
- new net ~{TXE}: H1.3, RN3.3 (R3.1)
- new net ~{WAKEUP}: H1.17, R4.2
- new net ~{WR}: H1.39, RN3.6 (R6.1)
- no-connect marks 0 -> 7
Other:
- note added: "Near pins 23, 26"
- moved on the sheet: U1, U2, U3
